Commit message: Right wheels rotate opposite direction to adjust to the real spur robot's config

File: spur_description/urdf/spur.urdf.xacro (robot description, xacro)
@@ -77,7 +77,7 @@
     <xacro:gazebo_link name="${suffix}_wheel_link"  color="Gray" />
   </xacro:macro>
-  <xacro:macro name="odom_wheel_rotate" params="suffix">
+  <xacro:macro name="odom_wheel_rotate" params="suffix rot_axis">
     <joint name="${suffix}_rotation_joint" type="revolute">
-      <axis xyz="0 0 1" />
+      <axis xyz="0 0 ${rot_axis}" />
       <limit lower="${-90*M_PI/180.0}" upper="${90*M_PI/180.0}" effort="300" velocity="1"/>
       <dynamics damping="50.0" friction="1.0" />
@@ -110,6 +110,6 @@
     <xacro:gazebo_link name="${suffix}_rotation_link"  color="LightGray" />
   </xacro:macro>
-  <xacro:macro name="odom_wheel" params="suffix *origin">
-    <xacro:odom_wheel_rotate suffix="${suffix}" />
+  <xacro:macro name="odom_wheel" params="suffix *origin rot_axis">
+    <xacro:odom_wheel_rotate suffix="${suffix}" rot_axis="${rot_axis}" />
     <xacro:odom_wheel_schaft suffix="${suffix}" />
     <xacro:odom_wheel_tire parent="${suffix}" suffix="l" offset="${0.05-wheel_width/2}"  />
@@ -283,14 +283,14 @@
   </joint>
   <!-- odom base -->
-  <xacro:odom_wheel suffix="fl">
+  <xacro:odom_wheel suffix="fl" rot_axis="1">
     <origin xyz="${caster_offset_x} ${caster_offset_y} 0.0" rpy="0 0 0" />
   </xacro:odom_wheel>
-  <xacro:odom_wheel suffix="fr">
+  <xacro:odom_wheel suffix="fr" rot_axis="-1">
     <origin xyz="${caster_offset_x} -${caster_offset_y} 0.0" rpy="0 0 0" />
   </xacro:odom_wheel>
-  <xacro:odom_wheel suffix="bl">
+  <xacro:odom_wheel suffix="bl" rot_axis="1">
     <origin xyz="-${caster_offset_x} ${caster_offset_y} 0.0" rpy="0 0 0" />
   </xacro:odom_wheel>
-  <xacro:odom_wheel suffix="br">
+  <xacro:odom_wheel suffix="br" rot_axis="-1">
     <origin xyz="-${caster_offset_x} -${caster_offset_y} 0.0" rpy="0 0 0" />
   </xacro:odom_wheel>

Commit message: yet another interpretation of Right wheels rotate opposite direction to adjust to the real spur robot

File: spur_description/urdf/spur.urdf.xacro (robot description, xacro)
@@ -46,7 +46,7 @@
     <xacro:gazebo_link name="${parent}_wheel_tire_${suffix}_link"  color="Black" />
   </xacro:macro>
-  <xacro:macro name="odom_wheel_schaft" params="suffix">
+  <xacro:macro name="odom_wheel_schaft" params="suffix rot_axis">
     <joint name="${suffix}_wheel_joint" type="continuous">
-      <axis xyz="0 0 1" />
+      <axis xyz="0 0 ${rot_axis}" />
       <limit effort="100" velocity="10"/>
       <dynamics damping="10.0" friction="0.0" />
@@ -77,7 +77,7 @@
     <xacro:gazebo_link name="${suffix}_wheel_link"  color="Gray" />
   </xacro:macro>
-  <xacro:macro name="odom_wheel_rotate" params="suffix rot_axis">
+  <xacro:macro name="odom_wheel_rotate" params="suffix">
     <joint name="${suffix}_rotation_joint" type="revolute">
-      <axis xyz="0 0 ${rot_axis}" />
+      <axis xyz="0 0 1" />
       <limit lower="${-90*M_PI/180.0}" upper="${90*M_PI/180.0}" effort="300" velocity="1"/>
       <dynamics damping="50.0" friction="1.0" />
@@ -111,6 +111,6 @@
   </xacro:macro>
   <xacro:macro name="odom_wheel" params="suffix *origin rot_axis">
-    <xacro:odom_wheel_rotate suffix="${suffix}" rot_axis="${rot_axis}" />
-    <xacro:odom_wheel_schaft suffix="${suffix}" />
+    <xacro:odom_wheel_rotate suffix="${suffix}" />
+    <xacro:odom_wheel_schaft suffix="${suffix}" rot_axis="${rot_axis}" />
     <xacro:odom_wheel_tire parent="${suffix}" suffix="l" offset="${0.05-wheel_width/2}"  />
     <xacro:odom_wheel_tire parent="${suffix}" suffix="r" offset="-${0.05-wheel_width/2}" />

Commit message: [spur.urdf.xacro] fix link order base_footprint -> base_link

File: spur_description/urdf/spur.urdf.xacro (robot description, xacro)
@@ -277,8 +277,8 @@
   <xacro:gazebo_link name="base_link"  color="Black" />
   <link name="base_footprint" />
-  <joint name="base_to_footprint" type="fixed" >
-    <origin xyz="0 0 -0.190" rpy="0 0 0" />
-    <parent link="base_link"/>
-    <child link="base_footprint" />
+  <joint name="footprint_to_base" type="fixed" >
+    <origin xyz="0 0 0.190" rpy="0 0 0" />
+    <parent link="base_footprint"/>
+    <child link="base_link" />
   </joint>
   <!-- odom base -->

Commit message: Complete adjusting model to real robot

File: spur_description/urdf/spur.urdf.xacro (robot description, xacro)
@@ -79,5 +79,5 @@
   <xacro:macro name="odom_wheel_rotate" params="suffix">
     <joint name="${suffix}_rotation_joint" type="revolute">
-      <axis xyz="0 0 1" />
+      <axis xyz="0 0 -1" />
       <limit lower="${-90*M_PI/180.0}" upper="${90*M_PI/180.0}" effort="300" velocity="1"/>
       <dynamics damping="50.0" friction="1.0" />

Commit message: if you want to put urg upside down, do not change visual, but change origin

File: spur_description/urdf/spur.urdf.xacro (robot description, xacro)
@@ -307,5 +307,5 @@
     </inertial>
     <visual>
-      <origin xyz="0 0 0" rpy="3.14 0 0"/>
+      <origin xyz="0 0 0" rpy="0 0 0"/>
       <geometry>
       <!-- <cylinder length="${hokuyo_length}" radius="${hokuyo_radius}" /> -->
@@ -321,5 +321,5 @@
   </link>
   <joint name="laser_to_base" type="fixed">
-    <origin xyz="${caster_offset_x} 0 -0.05" rpy="0 0 0" />
+    <origin xyz="${caster_offset_x} 0 -0.05" rpy="3.14 0 0" />
     <parent link="base_link" />
     <child link="hokuyo_sensor_link"/>
