Commit message: Add Hokuyo link and its gazebo plugin

File: spur_description/urdf/spur.gazebo.xacro (robot description, xacro)
@@ -1,4 +1,8 @@
 <?xml version="1.0"?>
-<robot xmlns:xacro="http://www.ros.org/wiki/xacro">
+<robot
+       xmlns:controller="http://playerstage.sourceforge.net/gazebo/xmlschema/#controller"
+       xmlns:interface="http://playerstage.sourceforge.net/gazebo/xmlschema/#interface"
+       xmlns:sensor="http://playerstage.sourceforge.net/gazebo/xmlschema/#sensor"
+       xmlns:xacro="http://www.ros.org/wiki/xacro">
   <!-- ros_control plugin -->
   <gazebo>
@@ -28,3 +32,36 @@
     </transmission>
   </xacro:macro>
+  <!-- URG -->
+  <!-- http://answers.ros.org/question/44691/how-to-put-hokuyo-laser-sensor-on-p2os/?answer=44785#post-id-44785 -->
+  <gazebo reference="hokuyo_sensor_link">
+      <sensor type="ray" name="laser">
+        <pose>0 0 0 0 0 0</pose>
+        <visualize>true</visualize>
+        <update_rate>40</update_rate>
+        <ray>
+          <scan>
+            <horizontal>
+              <samples>720</samples>
+              <resolution>1</resolution>
+              <min_angle>-1.570796</min_angle>
+              <max_angle>1.570796</max_angle>
+            </horizontal>
+          </scan>
+          <range>
+            <min>0.1</min>
+            <max>4.0</max>
+            <resolution>0.01</resolution>
+          </range>
+          <noise>
+            <type>Gaussian</type>
+            <mean>0.0</mean>
+            <stddev>0.01</stddev>
+          </noise>
+        </ray>
+        <plugin name="hokuyo_node" filename="libgazebo_ros_laser.so">
+          <topicName>/spur/laser/scan</topicName>
+          <frameName>/hokuyo_sensor_link</frameName>
+        </plugin>
+    </sensor>
+  </gazebo>
 </robot>

File: spur_description/urdf/spur.urdf.xacro (robot description, xacro)
@@ -18,4 +18,7 @@
   <property name="caster_offset_y" value="0.15" />
   <property name="caster_offset_z" value="0.14" />
+  <!-- Hokuyo https://www.hokuyo-aut.jp/02sensor/07scanner/urg_04lx.html -->
+  <property name="hokuyo_length" value="0.07" />
+  <property name="hokuyo_radius" value="0.043" /> <!-- Because max surface area of Hokuyo laser is not cylindrical, this isn't accurate, which shouldn't matter. -->
   <!-- wheel -->
   <xacro:macro name="odom_wheel_tire" params="parent suffix offset">
@@ -295,4 +298,31 @@
     <origin xyz="-${caster_offset_x} -${caster_offset_y} 0.0" rpy="0 0 0" />
   </xacro:odom_wheel>
+  <!-- URG -->
+  <!-- http://answers.ros.org/question/44691/how-to-put-hokuyo-laser-sensor-on-p2os/?answer=44785#post-id-44785 -->
+  <link name="hokuyo_sensor_link" type="laser">
+    <inertial>
+      <mass value="0.5" />
+      <origin xyz="0 0 0" />
+      <inertia ixx="0.3"  ixy="0.3"  ixz="0.3" iyy="0.3"  iyz="0.3"  izz="0.3" />
+    </inertial>
+    <visual>
+      <origin xyz="0 0 0" rpy="3.14 0 0"/>
+      <geometry>
+      <!-- <cylinder length="${hokuyo_length}" radius="${hokuyo_radius}" /> -->
+        <mesh filename="package://gazebo_plugins/test/multi_robot_scenario/meshes/laser/hokuyo.dae"/>
+      </geometry>
+     </visual>
+     <collision>
+       <origin xyz="0 0 0" rpy="0 0 0"/>
+       <geometry>
+         <cylinder length="${hokuyo_length}" radius="${hokuyo_radius}" />
+       </geometry>
+     </collision>
+  </link>
+  <joint name="laser_to_base" type="fixed">
+    <origin xyz="${caster_offset_x} 0 -0.05" rpy="0 0 0" />
+    <parent link="base_link" />
+    <child link="hokuyo_sensor_link"/>
+  </joint>
   <!-- arm -->
   <xacro:arm_links prefix="rarm" reflect="1" />

Commit message: update description, update inertia, effor

File: spur_description/urdf/spur.gazebo.xacro (robot description, xacro)
@@ -19,11 +19,30 @@
     </plugin>
   </gazebo>
-  <xacro:macro name="gazebo_link" params="name color">
+  <xacro:macro name="gazebo_tire_link" params="name color">
     <gazebo reference="${name}">
       <material>Gazebo/${color}</material>
-      <mu1 value="1.0" />
-      <mu2 value="1.0" />
-      <kp value="10000000.0" />
-      <kd value="1.0" />
+      <kp>500000.0</kp>
+      <kd>10.0</kd>
+      <mu1>10.0</mu1>
+      <mu2>10.0</mu2>
+      <fdir1>1 0 0</fdir1>
+      <minDepth>0.003</minDepth>
+    </gazebo>
+  </xacro:macro>
+  <xacro:macro name="gazebo_base_link" params="name color">
+    <gazebo reference="${name}">
+      <material>Gazebo/${color}</material>
+      <kp>1000000.0</kp>
+      <kd>10.0</kd>
+      <mu1>0.1</mu1>
+      <mu2>0.1</mu2>
+      <fdir1>1 0 0</fdir1>
+      <maxVel>10.0</maxVel>
+      <minDepth>0.0005</minDepth>
+    </gazebo>
+  </xacro:macro>
+  <xacro:macro name="gazebo_arm_link" params="name color">
+    <gazebo reference="${name}">
+      <material>Gazebo/${color}</material>
     </gazebo>
   </xacro:macro>

File: spur_description/urdf/spur.urdf.xacro (robot description, xacro)
@@ -32,6 +32,8 @@
         <mass value="1.0" />
         <origin xyz="0 0 0" />
-        <inertia  ixx="1.0" ixy="0.0" ixz="0.0"
-                  iyy="1.0" iyz="0.0" izz="1.0" />
+        <!-- <inertia  ixx="${((wheel_radius * wheel_radius / 4.0 ) + (wheel_width * wheel_width / 12.0 )) * 1.0}" ixy="0.0" ixz="0.0" -->
+        <!--           iyy="${((wheel_radius * wheel_radius / 4.0 ) + (wheel_width * wheel_width / 12.0 )) * 1.0}" iyz="0.0" -->
+        <!--           izz="${wheel_radius * wheel_radius / 2.0 * 1.0}" /> -->
+        <inertia ixx="0.1" ixy="0.0" ixz="0.0" iyy="0.1" iyz="0.0" izz="0.1"/>
       </inertial>
       <visual>
@@ -47,11 +49,11 @@
       </collision>
     </link>
-    <xacro:gazebo_link name="${parent}_wheel_tire_${suffix}_link"  color="Black" />
+    <xacro:gazebo_tire_link name="${parent}_wheel_tire_${suffix}_link"  color="Black" />
   </xacro:macro>
   <xacro:macro name="odom_wheel_schaft" params="suffix rot_axis">
     <joint name="${suffix}_wheel_joint" type="continuous">
       <axis xyz="0 0 ${rot_axis}" />
-      <limit effort="100" velocity="10"/>
-      <dynamics damping="10.0" friction="0.0" />
+      <limit effort="8.3" velocity="50"/> <!--  8.3 N/m ?? 45rpm -> 4.71 rad/s-->
+      <dynamics damping="0.0" friction="0.0" />
       <origin xyz="0 0 -${caster_offset_z}" rpy="-${M_PI/2} 0 0" />
       <parent link="${suffix}_rotation_link" />
@@ -61,8 +63,10 @@
     <link name="${suffix}_wheel_link">
       <inertial>
-        <mass value="1.0" />
+        <mass value="5.0" />
         <origin xyz="0 0 0" />
-        <inertia  ixx="1.0" ixy="0.0" ixz="0.0"
-                  iyy="1.0" iyz="0.0" izz="1.0" />
+        <!-- <inertia ixx="${((0.02 * 0.02 / 4.0 ) + (0.100 * 0.100 / 12.0)) * 5.0}" ixy="0.0" ixz="0.0" -->
+        <!--          iyy="${((0.02 * 0.02 / 4.0 ) + (0.100 * 0.100 / 12.0)) * 5.0}" iyz="0.0" -->
+        <!--          izz="${0.02 * 0.02 / 2.0 * 5.0}" /> -->
+        <inertia ixx="0.1" ixy="0.0" ixz="0.0" iyy="0.1" iyz="0.0" izz="0.1"/>
       </inertial>
       <visual>
@@ -74,15 +78,15 @@
       <collision>
         <geometry>
-          <cylinder length="0.100" radius="0.02"/>
-        </geometry>
-      </collision>
-    </link>
-    <xacro:gazebo_link name="${suffix}_wheel_link"  color="Gray" />
+          <cylinder length="${0.100 - wheel_width*2 - 0.01}" radius="0.02"/> <!-- avoid collision to tire -->
+        </geometry>
+      </collision>
+    </link>
+    <xacro:gazebo_tire_link name="${suffix}_wheel_link"  color="Grey" />
   </xacro:macro>
   <xacro:macro name="odom_wheel_rotate" params="suffix">
     <joint name="${suffix}_rotation_joint" type="revolute">
       <axis xyz="0 0 -1" />
-      <limit lower="${-90*M_PI/180.0}" upper="${90*M_PI/180.0}" effort="300" velocity="1"/>
-      <dynamics damping="50.0" friction="1.0" />
+      <limit lower="${-90*M_PI/180.0}" upper="${90*M_PI/180.0}" effort="50" velocity="4.71"/>
+      <dynamics damping="0.0" friction="0.0" />
       <xacro:insert_block name="origin" />
       <parent link="base_link"/>
@@ -93,10 +97,12 @@
       <inertial>
         <mass value="1.0" />
-        <origin xyz="0 0 0" />
-        <inertia  ixx="1.0" ixy="0.0" ixz="0.0"
-                  iyy="1.0" iyz="0.0" izz="1.0" />
-      </inertial>
-      <visual>
         <origin xyz="0 0 -${caster_offset_z/2}" rpy="0 0 0" />
+        <!-- <inertia  ixx="${((0.015 * 0.015 / 4.0 ) + (caster_offset_z * caster_offset_z / 12.0 )) * 1.0}" ixy="0.0" ixz="0.0" -->
+        <!--           iyy="${((0.015 * 0.015 / 4.0 ) + (caster_offset_z * caster_offset_z / 12.0 )) * 1.0}" iyz="0.0" -->
+        <!--           izz="${0.015 * 0.015 / 2.0 * 1.0}" /> -->
+        <inertia ixx="0.1" ixy="0.0" ixz="0.0" iyy="0.1" iyz="0.0" izz="0.1"/>
+      </inertial>
+      <visual>
+        <origin xyz="0 0 -${caster_offset_z/2}" rpy="0 0 0" />
         <geometry>
           <cylinder length="${caster_offset_z}" radius="0.015"/>
@@ -107,9 +113,9 @@
         <origin xyz="0 0 -${caster_offset_z/2}" rpy="0 0 0" />
         <geometry>
-          <cylinder length="${caster_offset_z}" radius="0.015"/>
-        </geometry>
-      </collision>
-    </link>
-    <xacro:gazebo_link name="${suffix}_rotation_link"  color="LightGray" />
+          <cylinder length="${caster_offset_z-0.05}" radius="0.015"/> <!-- avoid collision for wheel_schaft radius(0.02) -->
+        </geometry>
+      </collision>
+    </link>
+    <xacro:gazebo_base_link name="${suffix}_rotation_link"  color="White" />
   </xacro:macro>
   <xacro:macro name="odom_wheel" params="suffix *origin rot_axis">
@@ -123,8 +129,12 @@
     <link name="${name}">
       <inertial>
-        <mass value="1.0" />
+        <!-- <mass value="0.153" /> -->
         <xacro:insert_block name="origin" />
-        <inertia  ixx="1.0" ixy="0.0" ixz="0.0"
-                  iyy="1.0" iyz="0.0" izz="1.0" />
+        <!-- <inertia  ixx="${(0.0595/2*0.0595/2+0.0460/2*0.0460/2)/3*0.153}" ixy="0.0" ixz="0.0" -->
+        <!--           iyy="${(0.0460/2*0.0460/2+0.0290/2*0.0290/2)/3*0.153}" iyz="0.0" -->
+        <!--           izz="${(0.0290/2*0.0290/2+0.0595/2*0.0595/2)/3*0.153}" -->
+        <!--           /> -->
+        <mass value="1e-1" />
+        <inertia ixx="1e-2" ixy="0" ixz="0" iyy="1e-2" iyz="0" izz="1e-2" />
       </inertial>
       <visual>
@@ -138,17 +148,20 @@
         <xacro:insert_block name="origin" />
         <geometry>
-          <box size="0.029 0.0595 0.046" />
-        </geometry>
-      </collision>
-    </link>
-    <xacro:gazebo_link name="${name}"  color="Black" />
+          <box size="${0.029-0.001} ${0.0595-0.001} ${0.046-0.001}" />
+        </geometry>
+      </collision>
+    </link>
+    <xacro:gazebo_arm_link name="${name}"  color="Black" />
   </xacro:macro>
   <xacro:macro name="arm_link_element" params="name length" >
     <link name="${name}">
       <inertial>
-        <mass value="1.0" />
+        <!-- <mass value="0.1" /> -->
         <origin xyz="-${length/2 - 0.0145} 0 0" />
-        <inertia  ixx="1.0" ixy="0.0" ixz="0.0"
-                  iyy="1.0" iyz="0.0" izz="1.0" />
+        <!-- <inertia  ixx="${(0.029/2*0.029/2+0.005/2*0.005/2)/3*0.1}" ixy="0.0" ixz="0.0" -->
+        <!--           iyy="${(0.005/2*0.005/2+length/2*length/2)/3*0.1}" iyz="0.0" -->
+        <!--           izz="${(length/2*length/2+0.029/2*0.029/2)/3*0.1}" /> -->
+        <mass value="1e-5" />
+        <inertia ixx="1e-6" ixy="0" ixz="0" iyy="1e-6" iyz="0" izz="1e-6" />
       </inertial>
       <visual>
@@ -162,8 +175,8 @@
         <origin xyz="-${length/2 - 0.0145} 0 0"/>
         <geometry>
-          <box size="${length} 0.029 0.005" />
-        </geometry>
-      </collision>
-      <xacro:gazebo_link name="${name}"  color="LightGray" />
+          <box size="${length-0.06} 0.029 0.005" /> <!-- -0.06 to avoid self collision -->
+        </geometry>
+      </collision>
+      <xacro:gazebo_arm_link name="${name}"  color="White" />
     </link>
   </xacro:macro>
@@ -191,6 +204,6 @@
     <joint name="${name}_joint" type="revolute">
       <axis xyz="0 0 1" />
-      <limit lower="${-90*M_PI/180.0}" upper="${90*M_PI/180.0}" effort="300" velocity="1"/>
-      <dynamics damping="50.0" friction="1.0" />
+      <limit lower="${-90*M_PI/180.0}" upper="${90*M_PI/180.0}" effort="1" velocity="4.71"/>
+      <dynamics damping="0.0" friction="0.0" />
       <origin xyz="${joint_origin_xyz}" rpy="${joint_origin_rpy}" />
       <parent link="${parent}"/>
@@ -208,4 +221,5 @@
       <origin xyz="${link_origin_xyz}" rpy="${link_origin_rpy}" />
     </xacro:mx_106_link>
+    <xacro:gazebo_base_link name="${name}_link"  color="Black" />
   </xacro:macro>
   <xacro:macro name="arm_links" params="prefix reflect" >
@@ -239,14 +253,27 @@
                     link_origin_rpy="${M_PI/2} ${M_PI/2} 0" />
     <xacro:arm_joint parent="${prefix}_wrist_p_link" name="${prefix}_wrist_r"
-                     joint_origin_xyz="-0.05 0 0"
+                     joint_origin_xyz="-0.05 0.03 0"
                      joint_origin_rpy="-${M_PI/2} -${M_PI/2} 0" />
     <link name="${prefix}_wrist_r_link" >
       <inertial>
-        <mass value="1.0" />
         <origin xyz="0 0 0" />
-        <inertia  ixx="1.0" ixy="0.0" ixz="0.0"
-                  iyy="1.0" iyz="0.0" izz="1.0" />
-      </inertial>
-    </link>
+        <mass value="0.001" />
+        <inertia  ixx="${(0.001/2*0.001/2+0.001/2*0.001/2)/3*0.001}" ixy="0.0" ixz="0.0"
+                  iyy="${(0.001/2*0.001/2+0.001/2*0.001/2)/3*0.001}" iyz="0.0"
+                  izz="${(0.001/2*0.001/2+0.001/2*0.001/2)/3*0.001}" />
+      </inertial>
+      <visual>
+        <geometry>
+          <box size="0.02 0.02 0.02" />
+        </geometry>
+        <material name="DarkGrey" />
+      </visual>
+      <collision>
+        <geometry>
+          <box size="0.12 0.01 0.01" />
+        </geometry>
+      </collision>
+    </link>
+    <xacro:gazebo_arm_link name="${prefix}_wrist_r_link"  color="Black" />
     <xacro:arm_link_body name="${prefix}_elbow_p" length="0.2" >
       <origin xyz="0 0 0" rpy="0 0 0" />
@@ -261,6 +288,7 @@
       <mass value="10.0" />
       <origin xyz="0 0 0" />
-      <inertia  ixx="1.0" ixy="0.0" ixz="0.0"
-                iyy="1.0" iyz="0.0" izz="1.0" />
+      <inertia  ixx="${(base_width/2*base_width/2+base_height/2*base_height/2)/3*10.0}" ixy="0.0" ixz="0.0"
+                iyy="${(base_height/2*base_height/2+base_width/2*base_width/2)/3*10.0}"
+                iyz="0.0" izz="${(base_width/2*base_width/2+base_width/2*base_width/2)/3*10.0}" />
     </inertial>
     <visual>
@@ -278,5 +306,5 @@
     </collision>
   </link>
-  <xacro:gazebo_link name="base_link"  color="Black" />
+  <xacro:gazebo_base_link name="base_link"  color="Black" />
   <link name="base_footprint" />
   <joint name="footprint_to_base" type="fixed" >
@@ -299,22 +327,23 @@
   </xacro:odom_wheel>
   <!-- URG -->
-  <!-- http://answers.ros.org/question/44691/how-to-put-hokuyo-laser-sensor-on-p2os/?answer=44785#post-id-44785 -->
+  <!-- http://answers.ros.org/question/44691/how-to-put-hokuyo-laser-sensor-on-p2os/?answer=44785#post-id-44785   -->
   <link name="hokuyo_sensor_link" type="laser">
     <inertial>
-      <mass value="0.5" />
-      <origin xyz="0 0 0" />
-      <inertia ixx="0.3"  ixy="0.3"  ixz="0.3" iyy="0.3"  iyz="0.3"  izz="0.3" />
+      <mass value="0.160" />
+      <origin xyz="0 0 0.0" />
+      <inertia  ixx="${(0.05/2*0.05/2+0.07/2*0.07/2)/3*0.160}" ixy="0.0" ixz="0.0"
+                iyy="${(0.07/2*0.07/2+0.05/2*0.05/2)/3*0.160}" iyz="0.0"
+                izz="${(0.05/2*0.05/2+0.05/2*0.05/2)/3*0.160}" />
     </inertial>
     <visual>
       <origin xyz="0 0 0" rpy="0 0 0"/>
       <geometry>
-      <!-- <cylinder length="${hokuyo_length}" radius="${hokuyo_radius}" /> -->
         <mesh filename="package://gazebo_plugins/test/multi_robot_scenario/meshes/laser/hokuyo.dae"/>
       </geometry>
      </visual>
      <collision>
-       <origin xyz="0 0 0" rpy="0 0 0"/>
+       <origin xyz="0 0 0.0" />
        <geometry>
-         <cylinder length="${hokuyo_length}" radius="${hokuyo_radius}" />
+         <box size="0.05 0.05 0.07" />
        </geometry>
      </collision>
@@ -333,6 +362,6 @@
       <mass value="1.0" />
       <origin xyz="0 0 0.25" />
-      <inertia  ixx="1.0" ixy="0.0" ixz="0.0"
-                iyy="1.0" iyz="0.0" izz="1.0" />
+      <inertia  ixx="${(0.2/2*0.2/2+0.5/2*0.5/2)/3*1.0}" ixy="0.0" ixz="0.0"
+                iyy="${(0.5/2*0.5/2+0.1/2*0.1/2)/3*1.0}" iyz="0.0" izz="${(0.2/2*0.2/2+0.5/2*0.5/2)/3*1.0}" />
     </inertial>
     <visual>
@@ -350,5 +379,5 @@
     </collision>
   </link>
-  <xacro:gazebo_link name="body"  color="White" />
+  <xacro:gazebo_base_link name="body"  color="White" />
   <joint name="base_to_body" type="fixed" >
     <origin xyz="0 0 0.30" rpy="0 0 0" />
